File: it6302-remote-sense.sch (KiCad schematic (older format))
At the start: 31 parts, among them J1 POWER, J2 INTERNAL, J3 REMOTE, J4 SENSEOUT, J5 ENABLE, J6 LED, K1 RELAY-DPDT-EE2-SPLIT, K2 RELAY-DPDT-EE2-SPLIT, K3 RELAY-DPDT-EE2-SPLIT, Q1 3906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

Commit message: start layout
Parts:
- C1: footprint (none) -> libs:SMD-CP-6.3; symbol C -> CP
- D1, D2, D3: footprint (none) -> libs:SOT-23-DIODE
- J1: footprint (none) -> libs:JST-XH-2-PTH-TOP
- J2, J3, J4, J5, J6: footprint (none) -> libs:JST-XH-6-PTH-TOP
- K1, K2, K3: footprint (none) -> libs:RELAY-EE2-NU
- Q1, Q2, Q3: footprint (none) -> libs:SOT-23-BJT
- R1, R10, R11, R12, R13, R14, R15, R2, R3, R4, R5, R6, R7, R8, R9: footprint (none) -> libs:SMD-1608
Connections:
- net +12V: now also C1.+; no longer C1.1
- net COM: now also C1.-; no longer C1.2
Changed lines of the file:
@@
 LIBS:+15v
 LIBS:it6302-remote-sense-cache
-EELAYER 26 0
+EELAYER 25 0
 EELAYER END
 $Descr A4 11693 8268
@@
 F 0 "J3" H 2275 4050 50  0000 L CNN
 F 1 "REMOTE" H 2275 3950 50  0000 L CNN
-F 2 "" H 2150 4000 60  0000 C CNN
+F 2 "libs:JST-XH-6-PTH-TOP" H 2150 4000 60  0001 C CNN
 F 3 "" H 2150 4000 60  0000 C CNN
 	1    2050 4000
@@
 F 0 "J2" H 2275 3100 50  0000 L CNN
 F 1 "INTERNAL" H 2275 3000 50  0000 L CNN
-F 2 "" H 2150 3050 60  0000 C CNN
+F 2 "libs:JST-XH-6-PTH-TOP" H 2150 3050 60  0001 C CNN
 F 3 "" H 2150 3050 60  0000 C CNN
 	1    2050 3050
@@
 F 0 "J4" H 9625 3600 50  0000 L CNN
 F 1 "SENSEOUT" H 9625 3500 50  0000 L CNN
-F 2 "" H 9500 3550 60  0000 C CNN
+F 2 "libs:JST-XH-6-PTH-TOP" H 9500 3550 60  0001 C CNN
 F 3 "" H 9500 3550 60  0000 C CNN
 	1    9400 3550
@@
 F 0 "R4" V 6787 1600 50  0000 C CNN
 F 1 "1k" V 6696 1600 50  0000 C CNN
-F 2 "" H 7035 1590 60  0000 C CNN
+F 2 "libs:SMD-1608" H 7035 1590 60  0001 C CNN
 F 3 "" H 7035 1590 60  0000 C CNN
 	1    6900 1750
@@
 F 0 "K1" H 6950 1725 50  0000 L CNN
 F 1 "RELAY-DPDT-EE2-SPLIT" H 7050 1825 50  0001 C CNN
-F 2 "" H 7130 1560 50  0000 C CNN
+F 2 "libs:RELAY-EE2-NU" H 7130 1560 50  0001 C CNN
 F 3 "" H 7130 1560 50  0000 C CNN
 	1    7050 1600
@@
 F 0 "R5" V 6787 2250 50  0000 C CNN
 F 1 "1k" V 6696 2250 50  0000 C CNN
-F 2 "" H 7035 2240 60  0000 C CNN
+F 2 "libs:SMD-1608" H 7035 2240 60  0001 C CNN
 F 3 "" H 7035 2240 60  0000 C CNN
 	1    6900 2400
@@
 F 0 "K1" H 6950 2375 50  0000 L CNN
 F 1 "RELAY-DPDT-EE2-SPLIT" H 7050 2475 50  0001 C CNN
-F 2 "" H 7130 2210 50  0000 C CNN
+F 2 "libs:RELAY-EE2-NU" H 7130 2210 50  0001 C CNN
 F 3 "" H 7130 2210 50  0000 C CNN
 	2    7050 2250
@@
 F 0 "J6" H 9625 5050 50  0000 L CNN
 F 1 "LED" H 9625 4950 50  0000 L CNN
-F 2 "" H 9500 5000 60  0000 C CNN
+F 2 "libs:JST-XH-6-PTH-TOP" H 9500 5000 60  0001 C CNN
 F 3 "" H 9500 5000 60  0000 C CNN
 	1    9400 5000
@@
 F 0 "J5" H 2275 5050 50  0000 L CNN
 F 1 "ENABLE" H 2275 4950 50  0000 L CNN
-F 2 "" H 2150 5000 60  0000 C CNN
+F 2 "libs:JST-XH-6-PTH-TOP" H 2150 5000 60  0001 C CNN
 F 3 "" H 2150 5000 60  0000 C CNN
 	1    2050 5000
@@
 F 0 "R9" V 6787 3100 50  0000 C CNN
 F 1 "1k" V 6696 3100 50  0000 C CNN
-F 2 "" H 7035 3090 60  0000 C CNN
+F 2 "libs:SMD-1608" H 7035 3090 60  0001 C CNN
 F 3 "" H 7035 3090 60  0000 C CNN
 	1    6900 3250
@@
 F 0 "K2" H 6950 3225 50  0000 L CNN
 F 1 "RELAY-DPDT-EE2-SPLIT" H 7050 3325 50  0001 C CNN
-F 2 "" H 7130 3060 50  0000 C CNN
+F 2 "libs:RELAY-EE2-NU" H 7130 3060 50  0001 C CNN
 F 3 "" H 7130 3060 50  0000 C CNN
 	1    7050 3100
@@
 F 0 "R10" V 6787 3750 50  0000 C CNN
 F 1 "1k" V 6696 3750 50  0000 C CNN
-F 2 "" H 7035 3740 60  0000 C CNN
+F 2 "libs:SMD-1608" H 7035 3740 60  0001 C CNN
 F 3 "" H 7035 3740 60  0000 C CNN
 	1    6900 3900
@@
 F 0 "K2" H 6950 3875 50  0000 L CNN
 F 1 "RELAY-DPDT-EE2-SPLIT" H 7050 3975 50  0001 C CNN
-F 2 "" H 7130 3710 50  0000 C CNN
+F 2 "libs:RELAY-EE2-NU" H 7130 3710 50  0001 C CNN
 F 3 "" H 7130 3710 50  0000 C CNN
 	2    7050 3750
@@
 F 0 "R14" V 6787 4600 50  0000 C CNN
 F 1 "1k" V 6696 4600 50  0000 C CNN
-F 2 "" H 7035 4590 60  0000 C CNN
+F 2 "libs:SMD-1608" H 7035 4590 60  0001 C CNN
 F 3 "" H 7035 4590 60  0000 C CNN
 	1    6900 4750
@@
 F 0 "Q3" H 5325 4900 50  0000 L CNN
 F 1 "3906" H 5325 4800 50  0000 L CNN
-F 2 "" H 5300 4850 60  0000 C CNN
+F 2 "libs:SOT-23-BJT" H 5300 4850 60  0001 C CNN
 F 3 "" H 5300 4850 60  0000 C CNN
 	1    5300 4850
@@
 F 0 "R12" V 4755 4700 50  0000 C CNN
 F 1 "10k" V 4664 4700 50  0000 C CNN
-F 2 "" H 4685 4690 60  0000 C CNN
+F 2 "libs:SMD-1608" H 4685 4690 60  0001 C CNN
 F 3 "" H 4685 4690 60  0000 C CNN
 	1    4550 4850
@@
 F 0 "R11" H 4982 4446 50  0000 R CNN
 F 1 "10k" H 4982 4355 50  0000 R CNN
-F 2 "" H 5185 4390 60  0000 C CNN
+F 2 "libs:SMD-1608" H 5185 4390 60  0001 C CNN
 F 3 "" H 5185 4390 60  0000 C CNN
 	1    5050 4550
@@
 F 0 "D3" H 5170 5229 50  0000 L CNN
 F 1 "4148" H 5170 5320 50  0000 L CNN
-F 2 "" H 5100 5250 60  0000 C CNN
+F 2 "libs:SOT-23-DIODE" H 5100 5250 60  0001 C CNN
 F 3 "" H 5100 5250 60  0000 C CNN
 	1    5100 5400
@@
 F 0 "K3" H 6950 4725 50  0000 L CNN
 F 1 "RELAY-DPDT-EE2-SPLIT" H 7050 4825 50  0001 C CNN
-F 2 "" H 7130 4560 50  0000 C CNN
+F 2 "libs:RELAY-EE2-NU" H 7130 4560 50  0001 C CNN
 F 3 "" H 7130 4560 50  0000 C CNN
 	1    7050 4600
@@
 F 0 "K3" V 5300 5172 50  0000 R CNN
 F 1 "RELAY-DPDT-EE2-SPLIT" H 5300 5475 50  0001 C CNN
-F 2 "" H 5380 5210 50  0000 C CNN
+F 2 "libs:RELAY-EE2-NU" H 5380 5210 50  0001 C CNN
 F 3 "" H 5380 5210 50  0000 C CNN
 	3    5300 5250
@@
 F 0 "R13" H 5532 4896 50  0000 R CNN
 F 1 "10k" H 5532 4805 50  0000 R CNN
-F 2 "" H 5735 4840 60  0000 C CNN
+F 2 "libs:SMD-1608" H 5735 4840 60  0001 C CNN
 F 3 "" H 5735 4840 60  0000 C CNN
 	1    5600 5000
@@
 F 0 "R15" V 6787 5250 50  0000 C CNN
 F 1 "1k" V 6696 5250 50  0000 C CNN
-F 2 "" H 7035 5240 60  0000 C CNN
+F 2 "libs:SMD-1608" H 7035 5240 60  0001 C CNN
 F 3 "" H 7035 5240 60  0000 C CNN
 	1    6900 5400
@@
 F 0 "K3" H 6950 5375 50  0000 L CNN
 F 1 "RELAY-DPDT-EE2-SPLIT" H 7050 5475 50  0001 C CNN
-F 2 "" H 7130 5210 50  0000 C CNN
+F 2 "libs:RELAY-EE2-NU" H 7130 5210 50  0001 C CNN
 F 3 "" H 7130 5210 50  0000 C CNN
 	2    7050 5250
@@
 F 0 "Q2" H 5325 3400 50  0000 L CNN
 F 1 "3906" H 5325 3300 50  0000 L CNN
-F 2 "" H 5300 3350 60  0000 C CNN
+F 2 "libs:SOT-23-BJT" H 5300 3350 60  0001 C CNN
 F 3 "" H 5300 3350 60  0000 C CNN
 	1    5300 3350
@@
 F 0 "R7" V 4755 3200 50  0000 C CNN
 F 1 "10k" V 4664 3200 50  0000 C CNN
-F 2 "" H 4685 3190 60  0000 C CNN
+F 2 "libs:SMD-1608" H 4685 3190 60  0001 C CNN
 F 3 "" H 4685 3190 60  0000 C CNN
 	1    4550 3350
@@
 F 0 "R6" H 4982 2946 50  0000 R CNN
 F 1 "10k" H 4982 2855 50  0000 R CNN
-F 2 "" H 5185 2890 60  0000 C CNN
+F 2 "libs:SMD-1608" H 5185 2890 60  0001 C CNN
 F 3 "" H 5185 2890 60  0000 C CNN
 	1    5050 3050
@@
 F 0 "D2" H 5170 3729 50  0000 L CNN
 F 1 "4148" H 5170 3820 50  0000 L CNN
-F 2 "" H 5100 3750 60  0000 C CNN
+F 2 "libs:SOT-23-DIODE" H 5100 3750 60  0001 C CNN
 F 3 "" H 5100 3750 60  0000 C CNN
 	1    5100 3900
@@
 F 0 "K2" V 5300 3672 50  0000 R CNN
 F 1 "RELAY-DPDT-EE2-SPLIT" H 5300 3975 50  0001 C CNN
-F 2 "" H 5380 3710 50  0000 C CNN
+F 2 "libs:RELAY-EE2-NU" H 5380 3710 50  0001 C CNN
 F 3 "" H 5380 3710 50  0000 C CNN
 	3    5300 3750
@@
 F 0 "R8" H 5532 3396 50  0000 R CNN
 F 1 "10k" H 5532 3305 50  0000 R CNN
-F 2 "" H 5735 3340 60  0000 C CNN
+F 2 "libs:SMD-1608" H 5735 3340 60  0001 C CNN
 F 3 "" H 5735 3340 60  0000 C CNN
 	1    5600 3500
@@
 F 0 "Q1" H 5325 1900 50  0000 L CNN
 F 1 "3906" H 5325 1800 50  0000 L CNN
-F 2 "" H 5300 1850 60  0000 C CNN
+F 2 "libs:SOT-23-BJT" H 5300 1850 60  0001 C CNN
 F 3 "" H 5300 1850 60  0000 C CNN
 	1    5300 1850
@@
 F 0 "R2" V 4755 1700 50  0000 C CNN
 F 1 "10k" V 4664 1700 50  0000 C CNN
-F 2 "" H 4685 1690 60  0000 C CNN
+F 2 "libs:SMD-1608" H 4685 1690 60  0001 C CNN
 F 3 "" H 4685 1690 60  0000 C CNN
 	1    4550 1850
@@
 F 0 "R1" H 4982 1446 50  0000 R CNN
 F 1 "10k" H 4982 1355 50  0000 R CNN
-F 2 "" H 5185 1390 60  0000 C CNN
+F 2 "libs:SMD-1608" H 5185 1390 60  0001 C CNN
 F 3 "" H 5185 1390 60  0000 C CNN
 	1    5050 1550
@@
 F 0 "D1" H 5170 2229 50  0000 L CNN
 F 1 "4148" H 5170 2320 50  0000 L CNN
-F 2 "" H 5100 2250 60  0000 C CNN
+F 2 "libs:SOT-23-DIODE" H 5100 2250 60  0001 C CNN
 F 3 "" H 5100 2250 60  0000 C CNN
 	1    5100 2400
@@
 F 0 "K1" V 5300 2172 50  0000 R CNN
 F 1 "RELAY-DPDT-EE2-SPLIT" H 5300 2475 50  0001 C CNN
-F 2 "" H 5380 2210 50  0000 C CNN
+F 2 "libs:RELAY-EE2-NU" H 5380 2210 50  0001 C CNN
 F 3 "" H 5380 2210 50  0000 C CNN
 	3    5300 2250
@@
 F 0 "R3" H 5532 1896 50  0000 R CNN
 F 1 "10k" H 5532 1805 50  0000 R CNN
-F 2 "" H 5735 1840 60  0000 C CNN
+F 2 "libs:SMD-1608" H 5735 1840 60  0001 C CNN
 F 3 "" H 5735 1840 60  0000 C CNN
 	1    5600 2000
@@
 F 0 "J1" H 2078 1701 50  0000 L CNN
 F 1 "POWER" H 2078 1610 50  0000 L CNN
-F 2 "" H 1950 1450 60  0000 C CNN
+F 2 "libs:JST-XH-2-PTH-TOP" H 1950 1450 60  0001 C CNN
 F 3 "" H 1950 1450 60  0000 C CNN
 	1    1850 1650
@@
 $EndComp
 $Comp
-L C C1
+L CP C1
 U 1 1 5887BFF9
 P 2200 1550
 F 0 "C1" H 2273 1496 50  0000 L CNN
 F 1 "10u" H 2273 1405 50  0000 L CNN
-F 2 "" H 2100 1700 60  0000 C CNN
+F 2 "libs:SMD-CP-6.3" H 2100 1700 60  0001 C CNN
 F 3 "" H 2100 1700 60  0000 C CNN
 	1    2200 1550
